File: PIANO/_autosave-PIANO.kicad_sch (KiCad schematic)
At the start: 32 parts, among them J2 USB_B_Micro, J4 22-23-2021, SW1 ON/OFF, SW2 RESET, U1 LF33_TO220, U2 ESP32-S2-SOLO, U3 Opamp_Dual, U4 Opamp_Dual

Commit message: external spkr2
Connections:
- net +5V: no longer J2.1 (VBUS)
- net Output: no longer U2.4 (GPIO4/TOUCH4/ADC1_CH3), U3.3 (+)
- net Spkr 2: now reaches U2.5 (GPIO5/TOUCH5/ADC1_CH4)
- new net Spkr 1: U2.4 (GPIO4/TOUCH4/ADC1_CH3), U3.3 (+)
Other:
- added sheet Ext_Spkr2 (Ext_Spkr2_sch.kicad_sch)
Changed lines of the file:
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@@
   )
   (no_connect (at 166.37 173.99))
+  (no_connect (at 166.37 163.83))
   (no_connect (at 189.23 44.45))
   (no_connect (at 173.99 41.91))
@@
   (no_connect (at 158.75 31.75))
   (no_connect (at 158.75 34.29))
-  (no_connect (at 72.39 45.72))
   (no_connect (at 72.39 48.26))
   (no_connect (at 72.39 50.8))
@@
     (stroke (width 0) (type default) (color 0 0 0 0))
   )
+  (wire (pts (xy 60.96 45.72) (xy 60.96 54.61))
+    (stroke (width 0) (type default) (color 0 0 0 0))
+  )
   (wire (pts (xy 265.43 121.92) (xy 265.43 123.19))
     (stroke (width 0) (type default) (color 0 0 0 0))
@@
     (stroke (width 0) (type default) (color 0 0 0 0))
   )
+  (wire (pts (xy 72.39 45.72) (xy 60.96 45.72))
+    (stroke (width 0) (type default) (color 0 0 0 0))
+  )
   (wire (pts (xy 46.99 134.62) (xy 49.53 134.62))
     (stroke (width 0) (type default) (color 0 0 0 0))
@@
     (stroke (width 0) (type default) (color 0 0 0 0))
   )
+  (wire (pts (xy 60.96 54.61) (xy 63.5 54.61))
+    (stroke (width 0) (type default) (color 0 0 0 0))
+  )
   (polyline (pts (xy 12.7 105.41) (xy 110.49 105.41))
     (stroke (width 0) (type default) (color 0 0 0 0))
@@
     (stroke (width 0) (type default) (color 0 0 0 0))
   )
-  (wire (pts (xy 166.37 163.83) (xy 168.91 163.83))
-    (stroke (width 0) (type default) (color 0 0 0 0))
-  )
   (wire (pts (xy 54.61 125.73) (xy 62.23 125.73))
-    (stroke (width 0) (type default) (color 0 0 0 0))
-  )
-  (wire (pts (xy 168.91 160.02) (xy 168.91 163.83))
     (stroke (width 0) (type default) (color 0 0 0 0))
   )
@@
     (effects (font (size 1.27 1.27)) (justify left bottom))
   )
-  (label "Output" (at 180.34 25.4 180)
+  (label "Spkr 1" (at 180.34 25.4 180)
     (effects (font (size 1.27 1.27)) (justify right bottom))
   )
@@
     (effects (font (size 1.27 1.27)) (justify left bottom))
   )
-  (label "Output" (at 58.42 62.23 0)
+  (label "Spkr 2" (at 63.5 54.61 0)
+    (effects (font (size 1.27 1.27)) (justify left bottom))
+  )
+  (label "Spkr 1" (at 58.42 62.23 0)
     (effects (font (size 1.27 1.27)) (justify left bottom))
   )
@@
     (pin "1")
     (pin "2")
-  )
-  (symbol (lib_id "power:+5V") (at 168.91 160.02 0) (unit 1)
-    (in_bom yes) (on_board yes) (fields_autoplaced)
-    (property "Reference" "#PWR0127" (id 0) (at 168.91 163.83 0)
-      (effects (font (size 1.27 1.27)) hide)
-    )
-    (property "Value" "+5V" (id 1) (at 168.91 154.94 0))
-    (property "Footprint" "" (id 2) (at 168.91 160.02 0)
-      (effects (font (size 1.27 1.27)) hide)
-    )
-    (property "Datasheet" "" (id 3) (at 168.91 160.02 0)
-      (effects (font (size 1.27 1.27)) hide)
-    )
-    (pin "1")
   )
   (symbol (lib_id "Device:Opamp_Dual") (at 203.2 27.94 0) (unit 1)
@@
     )
   )
+  (sheet (at 12.7 148.59) (size 35.56 49.53) (fields_autoplaced)
+    (stroke (width 0.1524) (type solid) (color 0 0 0 0))
+    (fill (color 0 0 0 0.0000))
+    (property "Sheet name" "Ext_Spkr2" (id 0) (at 12.7 147.8784 0)
+      (effects (font (size 1.27 1.27)) (justify left bottom))
+    )
+    (property "Sheet file" "Ext_Spkr2_sch.kicad_sch" (id 1) (at 12.7 198.7046 0)
+      (effects (font (size 1.27 1.27)) (justify left top))
+    )
+  )
   (sheet_instances
     (path "/" (page "1"))
     (path "/7f576ece-c9bc-4f26-b53f-08232bf521db" (page "2"))
+    (path "/dc0bff4d-a643-4c20-a45a-98139025b2e3" (page "3"))
   )
   (symbol_instances
@@
       (reference "#PWR0126") (unit 1) (value "GND") (footprint "")
     )
-    (path "/2b629de8-a7b0-4d67-9b54-0b345dff9c5a"
-      (reference "#PWR0127") (unit 1) (value "+5V") (footprint "")
-    )
     (path "/7f576ece-c9bc-4f26-b53f-08232bf521db/93e95753-b550-4032-9af7-012ce2fbe4f7"
