File: PIANO/PIANO.kicad_sch (KiCad schematic)
At the start: 32 parts, among them J2 USB_B_Micro, J4 22-23-2021, SW1 ON/OFF, SW2 RESET, U1 LF33_TO220, U2 ESP32-S2-SOLO, U3 Opamp_Dual, U4 Opamp_Dual

Commit message: need to final check
Parts:
- added unit 2 of U3
Connections:
- net +5V: now also U3.8 (V+)
- no-connect marks 27 -> 30
Changed lines of the file:
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@@
   (no_connect (at 166.37 173.99))
   (no_connect (at 166.37 163.83))
+  (no_connect (at 168.91 40.64))
+  (no_connect (at 168.91 45.72))
+  (no_connect (at 184.15 43.18))
   (no_connect (at 72.39 86.36))
   (no_connect (at 158.75 36.83))
@@
   )
   (wire (pts (xy 40.64 16.51) (xy 52.07 16.51))
+    (stroke (width 0) (type default) (color 0 0 0 0))
+  )
+  (wire (pts (xy 212.09 33.02) (xy 212.09 35.56))
     (stroke (width 0) (type default) (color 0 0 0 0))
   )
@@
     (pin "1")
   )
+  (symbol (lib_id "power:+5V") (at 212.09 33.02 0) (unit 1)
+    (in_bom yes) (on_board yes) (fields_autoplaced)
+    (property "Reference" "#PWR0146" (id 0) (at 212.09 36.83 0)
+      (effects (font (size 1.27 1.27)) hide)
+    )
+    (property "Value" "+5V" (id 1) (at 212.09 27.94 0))
+    (property "Footprint" "" (id 2) (at 212.09 33.02 0)
+      (effects (font (size 1.27 1.27)) hide)
+    )
+    (property "Datasheet" "" (id 3) (at 212.09 33.02 0)
+      (effects (font (size 1.27 1.27)) hide)
+    )
+    (pin "1")
+  )
   (symbol (lib_id "Regulator_Linear:LF33_TO220") (at 46.99 125.73 0) (unit 1)
     (in_bom yes) (on_board yes) (fields_autoplaced)
@@
     (pin "3")
   )
-  (symbol (lib_id "power:PWR_FLAG") (at 212.09 35.56 0) (unit 1)
-    (in_bom yes) (on_board yes) (fields_autoplaced)
-    (property "Reference" "#FLG0101" (id 0) (at 212.09 33.655 0)
-      (effects (font (size 1.27 1.27)) hide)
-    )
-    (property "Value" "PWR_FLAG" (id 1) (at 212.09 30.48 0))
-    (property "Footprint" "" (id 2) (at 212.09 35.56 0)
-      (effects (font (size 1.27 1.27)) hide)
-    )
-    (property "Datasheet" "~" (id 3) (at 212.09 35.56 0)
-      (effects (font (size 1.27 1.27)) hide)
-    )
-    (pin "1")
-  )
   (symbol (lib_id "power:+3.3V") (at 29.21 93.98 0) (unit 1)
     (in_bom yes) (on_board yes) (fields_autoplaced)
@@
     (pin "1")
     (pin "2")
+  )
+  (symbol (lib_id "Device:Opamp_Dual") (at 176.53 43.18 0) (unit 2)
+    (in_bom yes) (on_board yes) (fields_autoplaced)
+    (property "Reference" "U3" (id 0) (at 176.53 33.02 0))
+    (property "Value" "Opamp_Dual" (id 1) (at 176.53 35.56 0))
+    (property "Footprint" "" (id 2) (at 176.53 43.18 0)
+      (effects (font (size 1.27 1.27)) hide)
+    )
+    (property "Datasheet" "~" (id 3) (at 176.53 43.18 0)
+      (effects (font (size 1.27 1.27)) hide)
+    )
+    (pin "5")
+    (pin "6")
+    (pin "7")
   )
   (symbol (lib_id "Device:R") (at 255.27 121.92 180) (unit 1)
@@
   )
   (symbol_instances
-    (path "/a7ba6e8b-d7ce-46ac-9514-5333a48e318e"
-      (reference "#FLG0101") (unit 1) (value "PWR_FLAG") (footprint "")
-    )
     (path "/7f576ece-c9bc-4f26-b53f-08232bf521db/1406e16c-b05a-4789-95a1-f137eaf3c632"
       (reference "#FLG0104") (unit 1) (value "PWR_FLAG") (footprint "")
@@
       (reference "#PWR0145") (unit 1) (value "+5V") (footprint "")
     )
+    (path "/96af6ba3-a837-4819-9bcd-5465c7e79808"
+      (reference "#PWR0146") (unit 1) (value "+5V") (footprint "")
+    )
     (path "/7f05d072-22d9-4098-ad43-15fc4a4844a4"
       (reference "C1") (unit 1) (value "10 uF") (footprint "Capacitor_SMD:C_0805_2012Metric")
@@
       (reference "U3") (unit 1) (value "Opamp_Dual") (footprint "Library:SOIC127P600X175-8N")
     )
+    (path "/c7c466c3-e68b-4e4f-a736-198f354b4956"
+      (reference "U3") (unit 2) (value "Opamp_Dual") (footprint "")
+    )
     (path "/149bff05-5e4c-49ef-9543-dc3c92cf2fdc"

Commit message: Semi-Final Product
Pin headers added, traces cleaned up, and figured out some funky grounding issues.
Parts:
- J4: footprint Connector_PinHeader_1.00mm:PinHeader_1x02_P1.00mm_Vertical -> Connector_PinHeader_2.54mm:PinHeader_1x02_P2.54mm_Vertical
- U3: footprint (none) -> Library:SOIC127P600X175-8N
Changed lines of the file:
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@@
       (effects (font (size 1.27 1.27)) (justify right))
     )
-    (property "Footprint" "Connector_PinHeader_1.00mm:PinHeader_1x02_P1.00mm_Vertical" (id 2) (at 260.35 24.13 0)
+    (property "Footprint" "Connector_PinHeader_2.54mm:PinHeader_1x02_P2.54mm_Vertical" (id 2) (at 260.35 24.13 0)
       (effects (font (size 1.524 1.524)) (justify left) hide)
     )
@@
     (property "Reference" "U3" (id 0) (at 176.53 33.02 0))
     (property "Value" "Opamp_Dual" (id 1) (at 176.53 35.56 0))
-    (property "Footprint" "" (id 2) (at 176.53 43.18 0)
+    (property "Footprint" "Library:SOIC127P600X175-8N" (id 2) (at 176.53 43.18 0)
       (effects (font (size 1.27 1.27)) hide)
     )
@@
     )
     (path "/dfbdb43d-ada6-42ef-9c58-d3d66952f5cc/767298c4-636e-4e6c-a62b-48710c53182e"
-      (reference "J1") (unit 1) (value "640456-3") (footprint "Connector_PinHeader_1.00mm:PinHeader_1x03_P1.00mm_Vertical")
+      (reference "J1") (unit 1) (value "640456-3") (footprint "Connector_PinHeader_2.54mm:PinHeader_1x03_P2.54mm_Vertical")
     )
     (path "/0ccf3bde-866e-4231-b785-fc8e0833134f"
@@
     )
     (path "/76cec44e-1374-41e1-9e39-24281d608b83"
-      (reference "J4") (unit 1) (value "22-23-2021") (footprint "Connector_PinHeader_1.00mm:PinHeader_1x02_P1.00mm_Vertical")
+      (reference "J4") (unit 1) (value "22-23-2021") (footprint "Connector_PinHeader_2.54mm:PinHeader_1x02_P2.54mm_Vertical")
     )
     (path "/dfbdb43d-ada6-42ef-9c58-d3d66952f5cc/26690c74-9ef1-4714-99af-adaf729b4b1e"
-      (reference "J5") (unit 1) (value "640456-3") (footprint "Connector_PinHeader_1.00mm:PinHeader_1x03_P1.00mm_Vertical")
+      (reference "J5") (unit 1) (value "640456-3") (footprint "Connector_PinHeader_2.54mm:PinHeader_1x03_P2.54mm_Vertical")
     )
     (path "/dfbdb43d-ada6-42ef-9c58-d3d66952f5cc/93a17808-eb11-4e49-9865-233fcfc7508c"
-      (reference "J6") (unit 1) (value "640456-3") (footprint "Connector_PinHeader_1.00mm:PinHeader_1x03_P1.00mm_Vertical")
+      (reference "J6") (unit 1) (value "640456-3") (footprint "Connector_PinHeader_2.54mm:PinHeader_1x03_P2.54mm_Vertical")
     )
     (path "/7f576ece-c9bc-4f26-b53f-08232bf521db/e9fcf1aa-31df-491c-8bb3-039d180f20f1"
@@
     )
     (path "/c7c466c3-e68b-4e4f-a736-198f354b4956"
-      (reference "U3") (unit 2) (value "Opamp_Dual") (footprint "")
+      (reference "U3") (unit 2) (value "Opamp_Dual") (footprint "Library:SOIC127P600X175-8N")
     )
     (path "/149bff05-5e4c-49ef-9543-dc3c92cf2fdc"
