File: PIANO/PIANO.kicad_sch (KiCad schematic)
At the start: 32 parts, among them J2 USB_B_Micro, J4 22-23-2021, SW1 ON/OFF, SW2 RESET, U1 LF33_TO220, U2 ESP32-S2-SOLO, U3 Opamp_Dual, U4 Opamp_Dual

Commit message: fixed most things
Parts:
- added J10, J11, J12, J13, J7, J8, J9: Conn_01x01_Female, Connector_PinHeader_2.54mm:PinHeader_1x01_P2.54mm_Vertical, symbol Connector:Conn_01x01_Female
Connections:
- net +3V3: now also J9.1 (Pin_1)
- net IO0 renamed RESET
- net Spkr 1 renamed SPKR_T
- net SPKR_T: now also J10.1 (Pin_1)
- new net 5V: J8.1 (Pin_1)
- new net 9V: J7.1 (Pin_1)
- new net STRP1_T: J11.1 (Pin_1)
- new net STRP2_T: J12.1 (Pin_1)
- new net STRP3_T: J13.1 (Pin_1)
