File: PIANO/LED_STRIPS.kicad_sch (KiCad schematic)
At the start: 6 parts, among them J1 640456-3, J5 640456-3, J6 640456-3

Commit message: Semi-Final Product
Pin headers added, traces cleaned up, and figured out some funky grounding issues.
Parts:
- J1, J5, J6: footprint Connector_PinHeader_1.00mm:PinHeader_1x03_P1.00mm_Vertical -> Connector_PinHeader_2.54mm:PinHeader_1x03_P2.54mm_Vertical
Changed lines of the file:
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@@
       (effects (font (size 1.27 1.27)) (justify right))
     )
-    (property "Footprint" "Connector_PinHeader_1.00mm:PinHeader_1x03_P1.00mm_Vertical" (id 2) (at 92.71 40.64 0)
+    (property "Footprint" "Connector_PinHeader_2.54mm:PinHeader_1x03_P2.54mm_Vertical" (id 2) (at 92.71 40.64 0)
       (effects (font (size 1.524 1.524)) (justify left) hide)
     )
@@
       (effects (font (size 1.27 1.27)) (justify right))
     )
-    (property "Footprint" "Connector_PinHeader_1.00mm:PinHeader_1x03_P1.00mm_Vertical" (id 2) (at 49.53 40.64 0)
+    (property "Footprint" "Connector_PinHeader_2.54mm:PinHeader_1x03_P2.54mm_Vertical" (id 2) (at 49.53 40.64 0)
       (effects (font (size 1.524 1.524)) (justify left) hide)
     )
@@
       (effects (font (size 1.27 1.27)) (justify right))
     )
-    (property "Footprint" "Connector_PinHeader_1.00mm:PinHeader_1x03_P1.00mm_Vertical" (id 2) (at 134.62 39.37 0)
+    (property "Footprint" "Connector_PinHeader_2.54mm:PinHeader_1x03_P2.54mm_Vertical" (id 2) (at 134.62 39.37 0)
       (effects (font (size 1.524 1.524)) (justify left) hide)
     )

Commit message: fixed most things
Connections:
- net Strip1 renamed STRP1_T
- net Strip2 renamed STRP2_T
- net Strip3 renamed STRP3_T
Changed lines of the file:
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@@
 (kicad_sch (version 20211123) (generator eeschema)
   (paper "A4")
+  (junction (at 39.37 26.67) (diameter 0) (color 0 0 0 0)
+  )
   (junction (at 39.37 43.18) (diameter 0) (color 0 0 0 0)
   )
+  (junction (at 82.55 26.67) (diameter 0) (color 0 0 0 0)
+  )
+  (junction (at 124.46 26.67) (diameter 0) (color 0 0 0 0)
+  )
   (junction (at 82.55 43.18) (diameter 0) (color 0 0 0 0)
   )
@@
     (stroke (width 0) (type default) (color 0 0 0 0))
   )
+  (wire (pts (xy 39.37 26.67) (xy 39.37 43.18))
+    (stroke (width 0) (type default) (color 0 0 0 0))
+  )
   (wire (pts (xy 82.55 43.18) (xy 95.25 43.18))
     (stroke (width 0) (type default) (color 0 0 0 0))
@@
     (stroke (width 0) (type default) (color 0 0 0 0))
   )
-  (wire (pts (xy 39.37 35.56) (xy 39.37 43.18))
+  (wire (pts (xy 39.37 21.59) (xy 39.37 26.67))
+    (stroke (width 0) (type default) (color 0 0 0 0))
+  )
+  (wire (pts (xy 82.55 26.67) (xy 87.63 26.67))
     (stroke (width 0) (type default) (color 0 0 0 0))
   )
@@
     (stroke (width 0) (type default) (color 0 0 0 0))
   )
+  (wire (pts (xy 39.37 26.67) (xy 41.91 26.67))
+    (stroke (width 0) (type default) (color 0 0 0 0))
+  )
   (wire (pts (xy 35.56 54.61) (xy 35.56 59.69))
     (stroke (width 0) (type default) (color 0 0 0 0))
@@
     (stroke (width 0) (type default) (color 0 0 0 0))
   )
-  (wire (pts (xy 124.46 34.29) (xy 124.46 41.91))
+  (wire (pts (xy 124.46 21.59) (xy 124.46 26.67))
     (stroke (width 0) (type default) (color 0 0 0 0))
   )
@@
     (stroke (width 0) (type default) (color 0 0 0 0))
   )
+  (wire (pts (xy 124.46 26.67) (xy 127 26.67))
+    (stroke (width 0) (type default) (color 0 0 0 0))
+  )
   (wire (pts (xy 52.07 35.56) (xy 52.07 40.64))
     (stroke (width 0) (type default) (color 0 0 0 0))
   )
-  (wire (pts (xy 82.55 35.56) (xy 82.55 43.18))
+  (wire (pts (xy 82.55 21.59) (xy 82.55 26.67))
     (stroke (width 0) (type default) (color 0 0 0 0))
   )
@@
     (stroke (width 0) (type default) (color 0 0 0 0))
   )
-  (label "Strip2" (at 82.55 35.56 180)
-    (effects (font (size 1.27 1.27)) (justify right bottom))
-  )
-  (label "Strip1" (at 39.37 35.56 180)
-    (effects (font (size 1.27 1.27)) (justify right bottom))
-  )
-  (label "Strip3" (at 124.46 34.29 180)
-    (effects (font (size 1.27 1.27)) (justify right bottom))
+  (wire (pts (xy 82.55 26.67) (xy 82.55 43.18))
+    (stroke (width 0) (type default) (color 0 0 0 0))
+  )
+  (wire (pts (xy 124.46 26.67) (xy 124.46 41.91))
+    (stroke (width 0) (type default) (color 0 0 0 0))
+  )
+  (global_label "STRP2_T" (shape input) (at 87.63 26.67 0) (fields_autoplaced)
+    (effects (font (size 1.27 1.27)) (justify left))
+    (property "Intersheet References" "${INTERSHEET_REFS}" (id 0) (at 97.905 26.5906 0)
+      (effects (font (size 1.27 1.27)) (justify left) hide)
+    )
+  )
+  (global_label "STRP3_T" (shape input) (at 127 26.67 0) (fields_autoplaced)
+    (effects (font (size 1.27 1.27)) (justify left))
+    (property "Intersheet References" "${INTERSHEET_REFS}" (id 0) (at 137.275 26.5906 0)
+      (effects (font (size 1.27 1.27)) (justify left) hide)
+    )
+  )
+  (global_label "Strip3" (shape input) (at 124.46 21.59 180) (fields_autoplaced)
+    (effects (font (size 1.27 1.27)) (justify right))
+    (property "Intersheet References" "${INTERSHEET_REFS}" (id 0) (at 116.3621 21.5106 0)
+      (effects (font (size 1.27 1.27)) (justify right) hide)
+    )
+  )
+  (global_label "STRP1_T" (shape input) (at 41.91 26.67 0) (fields_autoplaced)
+    (effects (font (size 1.27 1.27)) (justify left))
+    (property "Intersheet References" "${INTERSHEET_REFS}" (id 0) (at 52.185 26.5906 0)
+      (effects (font (size 1.27 1.27)) (justify left) hide)
+    )
+  )
+  (global_label "Strip1" (shape input) (at 39.37 21.59 180) (fields_autoplaced)
+    (effects (font (size 1.27 1.27)) (justify right))
+    (property "Intersheet References" "${INTERSHEET_REFS}" (id 0) (at 31.2721 21.5106 0)
+      (effects (font (size 1.27 1.27)) (justify right) hide)
+    )
+  )
+  (global_label "Strip2" (shape input) (at 82.55 21.59 180) (fields_autoplaced)
+    (effects (font (size 1.27 1.27)) (justify right))
+    (property "Intersheet References" "${INTERSHEET_REFS}" (id 0) (at 74.4521 21.5106 0)
+      (effects (font (size 1.27 1.27)) (justify right) hide)
+    )
   )
   (symbol (lib_id "power:GND") (at 137.16 48.26 0) (unit 1)
@@
   )
   (symbol (lib_id "power:+5V") (at 137.16 34.29 0) (unit 1)
-    (in_bom yes) (on_board yes) (fields_autoplaced)
+    (in_bom yes) (on_board yes)
     (property "Reference" "#PWR0145" (id 0) (at 137.16 38.1 0)
       (effects (font (size 1.27 1.27)) hide)
     )
-    (property "Value" "+5V" (id 1) (at 137.16 29.21 0))
+    (property "Value" "+5V" (id 1) (at 137.16 30.48 0))
     (property "Footprint" "" (id 2) (at 137.16 34.29 0)
       (effects (font (size 1.27 1.27)) hide)
@@
   )
   (symbol (lib_id "power:+5V") (at 52.07 35.56 0) (unit 1)
-    (in_bom yes) (on_board yes) (fields_autoplaced)
+    (in_bom yes) (on_board yes)
     (property "Reference" "#PWR0140" (id 0) (at 52.07 39.37 0)
       (effects (font (size 1.27 1.27)) hide)
     )
-    (property "Value" "+5V" (id 1) (at 52.07 30.48 0))
+    (property "Value" "+5V" (id 1) (at 52.07 31.75 0))
     (property "Footprint" "" (id 2) (at 52.07 35.56 0)
       (effects (font (size 1.27 1.27)) hide)
@@
   )
   (symbol (lib_id "power:+5V") (at 95.25 35.56 0) (unit 1)
-    (in_bom yes) (on_board yes) (fields_autoplaced)
+    (in_bom yes) (on_board yes)
     (property "Reference" "#PWR0131" (id 0) (at 95.25 39.37 0)
       (effects (font (size 1.27 1.27)) hide)
     )
-    (property "Value" "+5V" (id 1) (at 95.25 30.48 0))
+    (property "Value" "+5V" (id 1) (at 95.25 31.75 0))
     (property "Footprint" "" (id 2) (at 95.25 35.56 0)
       (effects (font (size 1.27 1.27)) hide)
