File: PIANO/PIANO.kicad_pcb (KiCad board)
At the start: 2 copper layers, 101.6 x 63.5 mm, 45 parts, among them J1 640456-3, J2 USB_B_Micro, J3 Barrel_Jack_Switch, J4 22-23-2021, J5 640456-3, J6 640456-3, SW1 ON/OFF, SW2 RESET, U1 LF33_TO220, U2 ESP32-S2-SOLO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

Commit message: added pos/neg
Parts:
- added J1: Conn_01x02_Male, Connector_PinHeader_2.54mm:PinHeader_1x02_P2.54mm_Vertical, F.Cu at (91.7, 94.1)
- J1, J5, J6: footprint Connector_PinHeader_2.54mm:PinHeader_1x03_P2.54mm_Vertical -> Connector_PinHeader_1.00mm:PinHeader_1x03_P1.00mm_Vertical
- J4: footprint Connector_PinHeader_2.54mm:PinHeader_1x02_P2.54mm_Vertical -> Connector_PinHeader_1.00mm:PinHeader_1x02_P1.00mm_Vertical
- moved L1 15.5 mm to (72.6, 100.3)
- moved J2 8.26 mm to (112.5, 116.4)
- moved J6 6.73 mm to (86.6, 70.6)
- moved C12 5.89 mm to (85.8, 74.7)
- moved J3 4.67 mm to (93.7, 109.0)
- moved J4 2.93 mm to (105.4, 106.2)
- moved J1 2.81 mm to (80.0, 70.6)
- moved C10 2.41 mm to (79.0, 74.4)
- moved C11 1.26 mm to (72.6, 74.2)
- moved J5 0.75 mm to (73.4, 70.6)
Routing:
- net GND: track 48.0 -> 60.6 mm, vias 12 -> 5
- net /D-: track 20.6 -> 13.7 mm
- net /D+: track 18.8 -> 12.6 mm
- net +5V: track 151.2 -> 148.8 mm
- net Net-(D4-Pad1): track 10.6 -> 8.58 mm
- net Net-(J4-Pad2): track 16.5 -> 15.2 mm
- net Net-(RV3-Pad2): track 40.6 -> 39.7 mm
- net /3 LED_STRIPS/Strip3: track 3.58 -> 4.36 mm
- removed copper zone on B.Cu, net GND
- removed copper zone on F.Cu, net GND
Other:
- board outline removed
- board text added: "+"
- board text added: "-"

Commit message: Pushing the Fiasco
Strange reversions cause Git algorithm sucks
Parts:
- J1, J5, J6: footprint Connector_PinHeader_1.00mm:PinHeader_1x03_P1.00mm_Vertical -> Connector_PinHeader_2.54mm:PinHeader_1x03_P2.54mm_Vertical
- J4: footprint Connector_PinHeader_1.00mm:PinHeader_1x02_P1.00mm_Vertical -> Connector_PinHeader_2.54mm:PinHeader_1x02_P2.54mm_Vertical
- moved J6 42.3 mm to (128.0, 79.0)
- moved J2 42.1 mm to (146.1, 142.0)
- moved C12 41.7 mm to (126.7, 82.7)
- moved J3 40.7 mm to (128.5, 130.1)
- moved J1 38.4 mm to (117.5, 79.0)
- moved J4 38.4 mm to (142.4, 116.5)
- moved C10 37.9 mm to (116.0, 82.7)
- moved C6 35.1 mm to (149.1, 99.8)
- moved RV1 35.1 mm to (148.4, 79.1)
- moved RV2 35.1 mm to (161.5, 79.0)
- moved U1 35.1 mm to (132.1, 102.4)
- moved U3 35.1 mm to (146.1, 109.0)
- moved C2 35.1 mm to (138.4, 100.5)
- moved C3 35.1 mm to (174.5, 107.5)
- moved C4 35.1 mm to (188.5, 99.1)
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Routing:
- net /D-: track 13.7 -> 29.8 mm
- net /D+: track 12.6 -> 28.0 mm
- net +5V: track 148.8 -> 162.6 mm
- net Net-(D4-Pad1): track 8.58 -> 19.0 mm
- net GND: track 60.6 -> 61.4 mm
- net Net-(RV3-Pad2): track 39.7 -> 38.9 mm
- net /3 LED_STRIPS/Strip3: track 4.36 -> 3.80 mm
- added copper zone on B.Cu, net GND
- added copper zone on F.Cu, net GND
Other:
- board outline added: 101.6 x 76.2 mm

Commit message: fixed most things
Parts:
- removed the J1 at (125.7, 102.5)
- added J10: Conn_01x01_Female, Connector_PinHeader_2.54mm:PinHeader_1x01_P2.54mm_Vertical, F.Cu at (186.8, 116.6)
- added J11: Conn_01x01_Female, Connector_PinHeader_2.54mm:PinHeader_1x01_P2.54mm_Vertical, F.Cu at (104.9, 72.5)
- added J12: Conn_01x01_Female, Connector_PinHeader_2.54mm:PinHeader_1x01_P2.54mm_Vertical, F.Cu at (115.1, 72.6)
- added J13: Conn_01x01_Female, Connector_PinHeader_2.54mm:PinHeader_1x01_P2.54mm_Vertical, F.Cu at (125.5, 72.5)
- added J7: Conn_01x01_Female, Connector_PinHeader_2.54mm:PinHeader_1x01_P2.54mm_Vertical, F.Cu at (122.2, 120.3)
- added J8: Conn_01x01_Female, Connector_PinHeader_2.54mm:PinHeader_1x01_P2.54mm_Vertical, F.Cu at (102.5, 120.3)
- added J9: Conn_01x01_Female, Connector_PinHeader_2.54mm:PinHeader_1x01_P2.54mm_Vertical, F.Cu at (135.6, 72.5)
- added REF**: MountingHole_3.2mm_M3, MountingHole:MountingHole_3.2mm_M3, F.Cu at (193.3, 140.2)
- added REF**: MountingHole_3.2mm_M3, MountingHole:MountingHole_3.2mm_M3, F.Cu at (101.9, 140.2)
- added REF**: MountingHole_3.2mm_M3, MountingHole:MountingHole_3.2mm_M3, F.Cu at (193.3, 73.3)
- C8: footprint Capacitor_SMD:C_1206_3216Metric -> Capacitor_SMD:C_1210_3225Metric
- moved J5 10.2 mm to (117.6, 79.1)
- moved C11 10.2 mm to (116.1, 82.7)
- moved C10 10.1 mm to (105.9, 82.7)
- moved J1 10.0 mm to (107.4, 79.0)
- moved U3 2.54 mm to (145.0, 106.7)
- moved C8 1.32 mm to (128.7, 111.4)
Connections:
- net +3V3 renamed 3.3V
- net +5V renamed 5V
- net +9V renamed 9V
- net /Spkr 1 renamed SPKR_T
- C10 pad 1: /3 LED_STRIPS/Strip1 -> Strip1
- C11 pad 1: /3 LED_STRIPS/Strip2 -> STRP2_T
- C12 pad 1: /3 LED_STRIPS/Strip3 -> STRP3_T
- J1 pad 2: /3 LED_STRIPS/Strip1 -> Strip1
- J5 pad 2: /3 LED_STRIPS/Strip2 -> STRP2_T
- J6 pad 2: /3 LED_STRIPS/Strip3 -> STRP3_T
- U2 pad 12: /Strip3 -> STRP3_T
- U2 pad 6: /Strip1 -> Strip1
- U2 pad 7: /Strip2 -> STRP2_T
Routing:
- net Strip1: track 0.00 -> 81.2 mm, vias 0 -> 2
- net STRP2_T: track 0.00 -> 73.4 mm, vias 0 -> 2
- net STRP3_T: track 0.00 -> 70.3 mm, vias 0 -> 2
- net SPKR_T: track 7.05 -> 48.1 mm, vias 0 -> 1
- net 5V: track 162.6 -> 180.6 mm
- net 9V: track 11.4 -> 18.9 mm
- net 3.3V: track 74.6 -> 81.0 mm
- net /3 LED_STRIPS/Strip3: track 3.80 -> 0.00 mm
- net /3 LED_STRIPS/Strip1: track 3.72 -> 0.00 mm
- net /3 LED_STRIPS/Strip2: track 3.64 -> 0.00 mm
- net Net-(J4-Pad2): track 15.0 -> 16.8 mm
- net Net-(R8-Pad2): track 11.9 -> 11.1 mm
- net GND: vias 5 -> 14
